Commit message: Fixed simulation issue

File: robot_ws/src/rover_description/urdf/suspension_left.xacro (robot description, xacro)
@@ -2,5 +2,5 @@
 <robot name="suspension_left" xmlns:xacro="http://www.ros.org/wiki/xacro">
     <xacro:macro name="suspension_left" params="">
-        <joint name="suspension_left_tree_root_joint" type="continuous">
+        <joint name="suspension_left_tree_root_joint" type="fixed">
             <origin xyz="${rocker_left_offset}" rpy="0.0 0.0 0.0"/>
             <parent link="chassis_link"/>

File: robot_ws/src/rover_description/urdf/suspension_right.xacro (robot description, xacro)
@@ -2,5 +2,5 @@
 <robot name="suspension_right" xmlns:xacro="http://www.ros.org/wiki/xacro">
     <xacro:macro name="suspension_right" params="">
-        <joint name="suspension_rigth_tree_root_joint" type="continuous">
+        <joint name="suspension_rigth_tree_root_joint" type="fixed">
             <origin xyz="${rocker_right_offset}" rpy="0.0 0.0 0.0"/>
             <parent link="chassis_link"/>

File: robot_ws/src/rover_description/urdf/wheel.xacro (robot description, xacro)
@@ -6,5 +6,7 @@
                 <origin xyz="${wheel_mass_center_xyz}" rpy="0.0 0.0 0.0"/>
                 <mass value="${wheel_mass}"/>
-                <inertia ixx="0.0" ixy="0.0" ixz="0.0" iyy="0.0" iyz="0.0" izz="0.0"/>
+                <inertia ixx="0.0004"   ixy="0.0"       ixz="0.0"
+                                        iyy="0.0002"    iyz="-0.0001"
+                                                        izz="0.0003"/>
             </inertial>
             <visual>

Commit message: Dynamics tag on joints

File: robot_ws/src/rover_description/urdf/suspension_left.xacro (robot description, xacro)
@@ -36,4 +36,5 @@
             <child link="bogie_pivot_left_link"/>
             <axis xyz="1.0 0.0 0.0"/>
+            <dynamics damping="0.0" friction="0.0"/>>
         </joint>
         <link name="bogie_pivot_left_link">
@@ -65,4 +66,5 @@
             <child link="drive_module_left_1_link"/>
             <axis xyz="0.0 0.0 1.0"/>
+            <dynamics damping="0.0" friction="0.0"/>
         </joint>
         <module_steerable
@@ -93,4 +95,5 @@
             <child link="bogie_1_wheel"/>
             <axis xyz="1.0 0.0 0.0"/>
+            <dynamics damping="0.5" friction="0.01"/>
         </joint>
         <wheel prefix="bogie_1" />
@@ -100,4 +103,5 @@
             <child link="bogie_2_wheel"/>
             <axis xyz="1.0 0.0 0.0"/>
+            <dynamics damping="0.5" friction="0.01"/>
         </joint>
         <wheel prefix="bogie_2" />
@@ -107,4 +111,5 @@
             <child link="bogie_3_wheel"/>
             <axis xyz="1.0 0.0 0.0"/>
+            <dynamics damping="0.5" friction="0.01"/>
         </joint>
         <wheel prefix="bogie_3" />

File: robot_ws/src/rover_description/urdf/suspension_right.xacro (robot description, xacro)
@@ -36,4 +36,5 @@
             <child link="bogie_pivot_right_link"/>
             <axis xyz="1.0 0.0 0.0"/>
+            <dynamics damping="0.0" friction="0.0"/>
         </joint>
         <link name="bogie_pivot_right_link">
@@ -65,4 +66,5 @@
             <child link="drive_module_right_3_link"/>
             <axis xyz="0.0 0.0 1.0"/>
+            <dynamics damping="0.0" friction="0.0"/>
         </joint>
         <module_steerable
@@ -79,4 +81,5 @@
             <child link="drive_module_right_4_link"/>
             <axis xyz="0.0 0.0 1.0"/>
+            <dynamics damping="0.0" friction="0.0"/>
         </joint>
         <module_steerable
@@ -93,4 +96,5 @@
             <child link="bogie_4_wheel"/>
             <axis xyz="1.0 0.0 0.0"/>
+            <dynamics damping="0.5" friction="0.01"/>
         </joint>
         <wheel prefix="bogie_4" />
@@ -100,4 +104,5 @@
             <child link="bogie_5_wheel"/>
             <axis xyz="1.0 0.0 0.0"/>
+            <dynamics damping="0.5" friction="0.01"/>
         </joint>
         <wheel prefix="bogie_5" />
@@ -107,4 +112,5 @@
             <child link="bogie_6_wheel"/>
             <axis xyz="1.0 0.0 0.0"/>
+            <dynamics damping="0.5" friction="0.01"/>
         </joint>
         <wheel prefix="bogie_6" />
