Commit message: New Parameters and right bogie tree ready. The new parameters fixes the error from main body's origin

File: robot_ws/src/rover_description/urdf/iteso_rover.xacro (robot description, xacro)
@@ -14,3 +14,4 @@
     <chassis />
     <suspension_left />
+    <suspension_right />
 </robot>

File: robot_ws/src/rover_description/urdf/iteso_rover_properies.xacro (robot description, xacro)
@@ -6,22 +6,25 @@
     <!-- Chassis properties -->
     <xacro:property name="chassis_mass" value="3.2015" />
-    <xacro:property name="chassis_mass_center_xyz" value="-0.0040 -0.0241 0.0604" />
+    <xacro:property name="chassis_mass_center_xyz" value="-0.0012 -0.0226 0.0618" />
     <!-- Suspension left -->
     <xacro:property name="rocker_left_mass" value="0.377" />
-    <xacro:property name="rocker_left_mass_center_xyz" value="0.0426 -0.026 0.0588" />
-    <xacro:property name="rocker_left_offset" value="0.15343 -0.07640 0.05432" />
+    <xacro:property name="rocker_left_mass_center_xyz" value="0.0426 -0.0588 -0.026" />
+    <xacro:property name="rocker_left_offset" value="0.15620 -0.07490 0.05507" />
     <!-- Suspension right -->
     <xacro:property name="rocker_right_mass" value="0.377" />
     <xacro:property name="rocker_right_mass_center_xyz" value="0.0649 0.0913 -0.0405" />
-    <xacro:property name="rocker_right_offset" value="-0.15343 -0.07640 0.05432" />
+    <xacro:property name="rocker_right_offset" value="-0.15620 -0.07490 0.05507" />
     <!-- Bogie pivot left -->
     <xacro:property name="bogie_pivot_left_mass" value="0.4062" />
     <xacro:property name="bogie_pivot_left_mass_center_xyz" value="0.2321 0.0187 0.063" />
-    <xacro:property name="bogie_pivot_left_offset" value="0.02470 0.18005 -0.06167" />
+    <xacro:property name="bogie_pivot_left_offset" value="0.0247 0.18007 -0.06163" />
     <!-- Bogie pivot right -->
+    <xacro:property name="bogie_pivot_right_mass" value="0.4062" />
+    <xacro:property name="bogie_pivot_right_mass_center_xyz" value="0.2321 0.0187 0.063" />
+    <xacro:property name="bogie_pivot_right_offset" value="-0.0247 0.18007 -0.06163" />
     <!-- Drive module left -->
-    <xacro:property name="drive_module_left_rpy" value="0.0 ${-PI/2}  ${-PI/2}" />
+    <xacro:property name="drive_module_left_rpy" value="0.0 0.0 0.0" />
     <xacro:property name="drive_module_left_mass" value="0.1978" />
-    <xacro:property name="drive_module_left_mass_center_xyz" value="-0.0425 0.0002 0.0381" />
+    <xacro:property name="drive_module_left_mass_center_xyz" value="-0.0392 -0.0273 0.0416" />
     <xacro:property name="drive_module_left_1_origin" value="0.02875 0 0" />
     <xacro:property name="drive_module_left_1_offset" value="0.07774 -0.21073 -0.15879" />
@@ -29,12 +32,24 @@
     <xacro:property name="drive_module_left_2_offset" value="0.05253 0.14854 -0.0981" />
     <!-- Drive module right -->
+    <xacro:property name="drive_module_right_rpy" value="0.0 0.0 0.0" />
+    <xacro:property name="drive_module_right_mass" value="0.1978" />
+    <xacro:property name="drive_module_right_mass_center_xyz" value="-0.0392 -0.0273 0.0416" />
+    <xacro:property name="drive_module_right_3_origin" value="-0.02875 0 0" />
+    <xacro:property name="drive_module_right_3_offset" value="-0.07774 -0.21073 -0.15879" />
+    <xacro:property name="drive_module_right_4_origin" value="-0.02874 0.0 0.0" />
+    <xacro:property name="drive_module_right_4_offset" value="-0.05253 0.14854 -0.0981" />
     <!-- Wheel -->
     <xacro:property name="wheel_mass" value="0.11466772" />
     <xacro:property name="wheel_mass_center_xyz" value="-0.0283157 0 -0.00034779" />
     <!-- Wheel left -->
+    <xacro:property name="wheel_left_rpy" value="0.0 0.0 0.0" />
     <xacro:property name="wheel_left_1_offset" value="0.03974 0.0 0.0" />
     <xacro:property name="wheel_left_2_offset" value="0.1185 -0.10696 -0.09649" />
     <xacro:property name="wheel_left_3_offset" value="0.03974 0.0 0.0" />
     <!-- Wheel right -->
+    <xacro:property name="wheel_right_rpy" value="0.0 0.0 ${PI}" />
+    <xacro:property name="wheel_left_4_offset" value="-0.03974 0.0 0.0" />
+    <xacro:property name="wheel_left_5_offset" value="-0.1185 -0.10696 -0.09649" />
+    <xacro:property name="wheel_left_6_offset" value="-0.03974 0.0 0.0" />
     <!-- Materials -->
     <material name="white">

File: robot_ws/src/rover_description/urdf/suspension_left.xacro (robot description, xacro)
@@ -12,7 +12,7 @@
                 <origin xyz="${rocker_left_mass_center_xyz}" rpy="0.0 0.0 0.0"/>
                 <mass value="${rocker_left_mass}"/>
-                <inertia    ixx="0.0077"    ixy="-0.0005"   ixz="0.0022"
-                                            iyy="0.0098"    iyz="-0.0003"
-                                                            izz="0.0015"/>
+                <inertia    ixx="0.0077"    ixy="-0.0012"   ixz="0.0"
+                                            iyy="0.0006"    iyz="-0.0002"
+                                                            izz="0.0078"/>
             </inertial>
             <visual>
@@ -41,7 +41,7 @@
                 <origin xyz="${bogie_pivot_left_mass_center_xyz}" rpy="0.0 0.0 0.0"/>
                 <mass value="${bogie_pivot_left_mass}"/>
-                <inertia    ixx="0.0684"    ixy="0.0038"    ixz="0.0"
-                                            iyy="0.0572"    iyz="-0.0028"
-                                                            izz="0.0425"/>
+                <inertia    ixx="0.0059"    ixy="-0.0002"    ixz="0.0002"
+                                            iyy="0.0014"    iyz="0.002"
+                                                            izz="0.0051"/>
             </inertial>
             <visual>
@@ -70,7 +70,7 @@
                 <origin xyz="${drive_module_left_mass_center_xyz}" rpy="${drive_module_left_rpy}"/>
                 <mass value="${drive_module_left_mass}"/>
-                <inertia    ixx="0.0"   ixy="0.0"   ixz="0.0"
-                                        iyy="0.0"   iyz="0.0"
-                                                    izz="0.0"/>
+                <inertia    ixx="0.0102"    ixy="0.0001"    ixz="0.0"
+                                            iyy="0.0063"    iyz="-0.0018"
+                                                            izz="0.0049"/>
             </inertial>
             <visual name="">
@@ -99,7 +99,7 @@
                 <origin xyz="${drive_module_left_mass_center_xyz}" rpy="${drive_module_left_rpy}"/>
                 <mass value="${drive_module_left_mass}"/>
-                <inertia    ixx="0.0"   ixy="0.0"   ixz="0.0"
-                                        iyy="0.0"   iyz="0.0"
-                                                    izz="0.0"/>
+                <inertia    ixx="0.0102"    ixy="0.0001"    ixz="0.0"
+                                            iyy="0.0063"    iyz="-0.0018"
+                                                            izz="0.0049"/>
             </inertial>
             <visual name="">
@@ -119,5 +119,5 @@
         </link>
         <joint name="wheel_1_joint" type="continuous">
-            <origin xyz="${wheel_left_1_offset}" rpy="0.0 0.0 0.0"/>
+            <origin xyz="${wheel_left_1_offset}" rpy="${wheel_left_rpy}"/>
             <parent link="drive_module_left_1_link"/>
             <child link="bogie_1_wheel"/>
@@ -126,5 +126,5 @@
         <wheel prefix="bogie_1" />
         <joint name="wheel_2_joint" type="continuous">
-            <origin xyz="${wheel_left_2_offset}" rpy="0.0 0.0 0.0"/>
+            <origin xyz="${wheel_left_2_offset}" rpy="${wheel_left_rpy}"/>
             <parent link="bogie_pivot_left_link"/>
             <child link="bogie_2_wheel"/>
@@ -133,5 +133,5 @@
         <wheel prefix="bogie_2" />
         <joint name="wheel_3_joint" type="continuous">
-            <origin xyz="${wheel_left_3_offset}" rpy="0.0 0.0 0.0"/>
+            <origin xyz="${wheel_left_3_offset}" rpy="${wheel_left_rpy}"/>
             <parent link="drive_module_left_2_link"/>
             <child link="bogie_3_wheel"/>

File: robot_ws/src/rover_description/urdf/suspension_right.xacro (robot description, xacro)
@@ -1,5 +1,5 @@
 <?xml version="1.0"?>
 <robot name="suspension_right" xmlns:xacro="http://www.ros.org/wiki/xacro">
-    <xacro:macro name="suspension_rigth" params="">
+    <xacro:macro name="suspension_right" params="">
         <joint name="suspension_rigth_tree_root_joint" type="continuous">
             <origin xyz="${rocker_right_offset}" rpy="0.0 0.0 0.0"/>
@@ -10,6 +10,6 @@
         <link name="rocker_right_link">
             <inertial>
-                <origin xyz="${rocker_left_mass_center_xyz}" rpy="0.0 0.0 0.0"/>
-                <mass value="${rocker_left_mass}"/>
+                <origin xyz="${rocker_right_mass_center_xyz}" rpy="0.0 0.0 0.0"/>
+                <mass value="${rocker_right_mass}"/>
                 <inertia    ixx="0.0077"    ixy="-0.0005"   ixz="0.0022"
                                             iyy="0.0098"    iyz="-0.0003"
@@ -25,5 +25,5 @@
             </visual>
             <collision>
-                <origin xyz="0.0 0.0 0.0" rpy="0.0 0.0 ${-PI/2}"/>
+                <origin xyz="0.0 0.0 0.0" rpy="0.0 0.0 0.0"/>
                 <geometry>
                     <mesh filename="package://rover_description/meshes/MirrorRocker.STL" scale="${SCALE_XYZ}"/>
@@ -31,8 +31,7 @@
             </collision>
         </link>
-        <!--
         <joint name="rocker_bogie_right" type="continuous">
-            <origin xyz="${bogie_pivot_left_offset}" rpy="0.0 0.0 0.0"/>
-            <parent link="rocker_left_link"/>
+            <origin xyz="${bogie_pivot_right_offset}" rpy="0.0 0.0 0.0"/>
+            <parent link="rocker_right_link"/>
             <child link="bogie_pivot_right_link"/>
             <axis xyz="1.0 0.0 0.0"/>
@@ -40,6 +39,6 @@
         <link name="bogie_pivot_right_link">
             <inertial>
-                <origin xyz="${bogie_pivot_left_mass_center_xyz}" rpy="0.0 0.0 0.0"/>
-                <mass value="${bogie_pivot_left_mass}"/>
+                <origin xyz="${bogie_pivot_right_mass_center_xyz}" rpy="0.0 0.0 0.0"/>
+                <mass value="${bogie_pivot_right_mass}"/>
                 <inertia    ixx="0.0684"    ixy="0.0038"    ixz="0.0"
                                             iyy="0.0572"    iyz="-0.0028"
@@ -49,5 +48,5 @@
                 <origin xyz="0.0 0.0 0.0" rpy="0.0 0.0 0.0"/>
                 <geometry>
-                    <mesh filename="package://rover_description/meshes/Bogie_pivot.STL" scale="${SCALE_XYZ}"/>
+                    <mesh filename="package://rover_description/meshes/MirrorBogie_pivot.STL" scale="${SCALE_XYZ}"/>
                 </geometry>
                 <material name="white">
@@ -57,9 +56,87 @@
                 <origin xyz="0.0 0.0 0.0" rpy="0.0 0.0 0.0"/>
                 <geometry>
-                    <mesh filename="package://rover_description/meshes/Bogie_pivot.STL" scale="${SCALE_XYZ}"/>
+                    <mesh filename="package://rover_description/meshes/MirrorBogie_pivot.STL" scale="${SCALE_XYZ}"/>
                 </geometry>
             </collision>
         </link>
-        -->
+        <joint name="bogie_drive_right_3" type="continuous">
+            <origin xyz="${drive_module_right_3_offset}" rpy="0.0 0.0 0.0"/>
+            <parent link="rocker_right_link"/>
+            <child link="drive_module_right_3_link"/>
+            <axis xyz="0.0 0.0 1.0"/>
+        </joint>
+        <link name="drive_module_right_3_link">
+            <inertial>
+                <origin xyz="${drive_module_right_mass_center_xyz}" rpy="${drive_module_right_rpy}"/>
+                <mass value="${drive_module_right_mass}"/>
+                <inertia    ixx="0.0102"    ixy="0.0001"    ixz="0.0"
+                                            iyy="0.0063"    iyz="-0.0018"
+                                                            izz="0.0049"/>
+            </inertial>
+            <visual name="">
+                <origin xyz="${drive_module_right_3_origin}" rpy="${drive_module_right_rpy}"/>
+                <geometry>
+                    <mesh filename="package://rover_description/meshes/MirrorDrive Module_steerable.STL" scale="${SCALE_XYZ}"/>
+                </geometry>
+                <material name="white">
+                </material>
+            </visual>
+            <collision>
+                <origin xyz="${drive_module_right_3_origin}" rpy="${drive_module_right_rpy}"/>
+                <geometry>
+                    <mesh filename="package://rover_description/meshes/MirrorDrive Module_steerable.STL" scale="${SCALE_XYZ}"/>
+                </geometry>
+            </collision>
+        </link>
+        <joint name="bogie_drive_right_4" type="continuous">
+            <origin xyz="${drive_module_right_4_offset}" rpy="0.0 0.0 0.0"/>
+            <parent link="bogie_pivot_right_link"/>
+            <child link="drive_module_right_4_link"/>
+            <axis xyz="0.0 0.0 1.0"/>
+        </joint>
+        <link name="drive_module_right_4_link">
+            <inertial>
+                <origin xyz="${drive_module_right_mass_center_xyz}" rpy="${drive_module_right_rpy}"/>
+                <mass value="${drive_module_right_mass}"/>
+                <inertia    ixx="0.0102"    ixy="0.0001"    ixz="0.0"
+                                            iyy="0.0063"    iyz="-0.0018"
+                                                            izz="0.0049"/>
+            </inertial>
+            <visual name="">
+                <origin xyz="${drive_module_right_3_origin}" rpy="${drive_module_right_rpy}"/>
+                <geometry>
+                    <mesh filename="package://rover_description/meshes/MirrorDrive Module_steerable.STL" scale="${SCALE_XYZ}"/>
+                </geometry>
+                <material name="white">
+                </material>
+            </visual>
+            <collision>
+                <origin xyz="${drive_module_right_3_origin}" rpy="${drive_module_right_rpy}"/>
+                <geometry>
+                    <mesh filename="package://rover_description/meshes/MirrorDrive Module_steerable.STL" scale="${SCALE_XYZ}"/>
+                </geometry>
+            </collision>
+        </link>
+        <joint name="wheel_4_joint" type="continuous">
+            <origin xyz="${wheel_left_4_offset}" rpy="${wheel_right_rpy}"/>
+            <parent link="drive_module_right_3_link"/>
+            <child link="bogie_4_wheel"/>
+            <axis xyz="1.0 0.0 0.0"/>
+        </joint>
+        <wheel prefix="bogie_4" />
+        <joint name="wheel_5_joint" type="continuous">
+            <origin xyz="${wheel_left_5_offset}" rpy="${wheel_right_rpy}"/>
+            <parent link="bogie_pivot_right_link"/>
+            <child link="bogie_5_wheel"/>
+            <axis xyz="1.0 0.0 0.0"/>
+        </joint>
+        <wheel prefix="bogie_5" />
+        <joint name="wheel_6_joint" type="continuous">
+            <origin xyz="${wheel_left_6_offset}" rpy="${wheel_right_rpy}"/>
+            <parent link="drive_module_right_4_link"/>
+            <child link="bogie_6_wheel"/>
+            <axis xyz="1.0 0.0 0.0"/>
+        </joint>
+        <wheel prefix="bogie_6" />
     </xacro:macro>
 </robot>
