Commit message: New macros

File: robot_ws/src/rover_description/urdf/iteso_rover.xacro (robot description, xacro)
@@ -11,4 +11,6 @@
     <!-- Wheel -->
     <xacro:include filename="$(find rover_description)/urdf/wheel.xacro" />
+    <!-- Module Steerable -->
+    <xacro:include filename="$(find rover_description)/urdf/drive_module_steerable.xacro"/>
     <!-- Macros calls -->
     <chassis />

File: robot_ws/src/rover_description/urdf/iteso_rover_properies.xacro (robot description, xacro)
@@ -49,7 +49,7 @@
     <!-- Wheel right -->
     <xacro:property name="wheel_right_rpy" value="0.0 0.0 ${PI}" />
-    <xacro:property name="wheel_left_4_offset" value="-0.03974 0.0 0.0" />
-    <xacro:property name="wheel_left_5_offset" value="-0.1185 -0.10696 -0.09649" />
-    <xacro:property name="wheel_left_6_offset" value="-0.03974 0.0 0.0" />
+    <xacro:property name="wheel_right_4_offset" value="-0.03974 0.0 0.0" />
+    <xacro:property name="wheel_right_5_offset" value="-0.1185 -0.10696 -0.09649" />
+    <xacro:property name="wheel_right_6_offset" value="-0.03974 0.0 0.0" />
     <!-- Materials -->
     <material name="white">

File: robot_ws/src/rover_description/urdf/suspension_left.xacro (robot description, xacro)
@@ -66,27 +66,12 @@
             <axis xyz="0.0 0.0 1.0"/>
         </joint>
-        <link name="drive_module_left_1_link">
-            <inertial>
-                <origin xyz="${drive_module_left_mass_center_xyz}" rpy="${drive_module_left_rpy}"/>
-                <mass value="${drive_module_left_mass}"/>
-                <inertia    ixx="0.0102"    ixy="0.0001"    ixz="0.0"
-                                            iyy="0.0063"    iyz="-0.0018"
-                                                            izz="0.0049"/>
-            </inertial>
-            <visual name="">
-                <origin xyz="${drive_module_left_1_origin}" rpy="${drive_module_left_rpy}"/>
-                <geometry>
-                    <mesh filename="package://rover_description/meshes/Drive Module_steerable.STL" scale="${SCALE_XYZ}"/>
-                </geometry>
-                <material name="white">
-                </material>
-            </visual>
-            <collision>
-                <origin xyz="${drive_module_left_1_origin}" rpy="${drive_module_left_rpy}"/>
-                <geometry>
-                    <mesh filename="package://rover_description/meshes/Drive Module_steerable.STL" scale="${SCALE_XYZ}"/>
-                </geometry>
-            </collision>
-        </link>
+        <module_steerable
+            name="drive_module_left_1_link"
+            mass="${drive_module_left_mass}"
+            mass_center="${drive_module_left_mass_center_xyz}"
+            origin_xyz="${drive_module_left_1_origin}"
+            origin_rpy="${drive_module_left_rpy}"
+            mesh_filename="package://rover_description/meshes/Drive Module_steerable.STL"
+        />
         <joint name="bogie_drive_left_2" type="continuous">
             <origin xyz="${drive_module_left_2_offset}" rpy="0.0 0.0 0.0"/>
@@ -95,27 +80,12 @@
             <axis xyz="0.0 0.0 1.0"/>
         </joint>
-        <link name="drive_module_left_2_link">
-            <inertial>
-                <origin xyz="${drive_module_left_mass_center_xyz}" rpy="${drive_module_left_rpy}"/>
-                <mass value="${drive_module_left_mass}"/>
-                <inertia    ixx="0.0102"    ixy="0.0001"    ixz="0.0"
-                                            iyy="0.0063"    iyz="-0.0018"
-                                                            izz="0.0049"/>
-            </inertial>
-            <visual name="">
-                <origin xyz="${drive_module_left_2_origin}" rpy="${drive_module_left_rpy}"/>
-                <geometry>
-                    <mesh filename="package://rover_description/meshes/Drive Module_steerable.STL" scale="${SCALE_XYZ}"/>
-                </geometry>
-                <material name="white">
-                </material>
-            </visual>
-            <collision>
-                <origin xyz="${drive_module_left_2_origin}" rpy="${drive_module_left_rpy}"/>
-                <geometry>
-                    <mesh filename="package://rover_description/meshes/Drive Module_steerable.STL" scale="${SCALE_XYZ}"/>
-                </geometry>
-            </collision>
-        </link>
+        <module_steerable
+            name="drive_module_left_2_link"
+            mass="${drive_module_left_mass}"
+            mass_center="${drive_module_left_mass_center_xyz}"
+            origin_xyz="${drive_module_left_2_origin}"
+            origin_rpy="${drive_module_left_rpy}"
+            mesh_filename="package://rover_description/meshes/Drive Module_steerable.STL"
+        />
         <joint name="wheel_1_joint" type="continuous">
             <origin xyz="${wheel_left_1_offset}" rpy="${wheel_left_rpy}"/>

File: robot_ws/src/rover_description/urdf/suspension_right.xacro (robot description, xacro)
@@ -66,27 +66,12 @@
             <axis xyz="0.0 0.0 1.0"/>
         </joint>
-        <link name="drive_module_right_3_link">
-            <inertial>
-                <origin xyz="${drive_module_right_mass_center_xyz}" rpy="${drive_module_right_rpy}"/>
-                <mass value="${drive_module_right_mass}"/>
-                <inertia    ixx="0.0102"    ixy="0.0001"    ixz="0.0"
-                                            iyy="0.0063"    iyz="-0.0018"
-                                                            izz="0.0049"/>
-            </inertial>
-            <visual name="">
-                <origin xyz="${drive_module_right_3_origin}" rpy="${drive_module_right_rpy}"/>
-                <geometry>
-                    <mesh filename="package://rover_description/meshes/MirrorDrive Module_steerable.STL" scale="${SCALE_XYZ}"/>
-                </geometry>
-                <material name="white">
-                </material>
-            </visual>
-            <collision>
-                <origin xyz="${drive_module_right_3_origin}" rpy="${drive_module_right_rpy}"/>
-                <geometry>
-                    <mesh filename="package://rover_description/meshes/MirrorDrive Module_steerable.STL" scale="${SCALE_XYZ}"/>
-                </geometry>
-            </collision>
-        </link>
+        <module_steerable
+            name="drive_module_right_3_link"
+            mass="${drive_module_right_mass}"
+            mass_center="${drive_module_right_mass_center_xyz}"
+            origin_xyz="${drive_module_right_4_origin}"
+            origin_rpy="${drive_module_right_rpy}"
+            mesh_filename="package://rover_description/meshes/MirrorDrive Module_steerable.STL"
+        />
         <joint name="bogie_drive_right_4" type="continuous">
             <origin xyz="${drive_module_right_4_offset}" rpy="0.0 0.0 0.0"/>
@@ -95,29 +80,14 @@
             <axis xyz="0.0 0.0 1.0"/>
         </joint>
-        <link name="drive_module_right_4_link">
-            <inertial>
-                <origin xyz="${drive_module_right_mass_center_xyz}" rpy="${drive_module_right_rpy}"/>
-                <mass value="${drive_module_right_mass}"/>
-                <inertia    ixx="0.0102"    ixy="0.0001"    ixz="0.0"
-                                            iyy="0.0063"    iyz="-0.0018"
-                                                            izz="0.0049"/>
-            </inertial>
-            <visual name="">
-                <origin xyz="${drive_module_right_3_origin}" rpy="${drive_module_right_rpy}"/>
-                <geometry>
-                    <mesh filename="package://rover_description/meshes/MirrorDrive Module_steerable.STL" scale="${SCALE_XYZ}"/>
-                </geometry>
-                <material name="white">
-                </material>
-            </visual>
-            <collision>
-                <origin xyz="${drive_module_right_3_origin}" rpy="${drive_module_right_rpy}"/>
-                <geometry>
-                    <mesh filename="package://rover_description/meshes/MirrorDrive Module_steerable.STL" scale="${SCALE_XYZ}"/>
-                </geometry>
-            </collision>
-        </link>
+        <module_steerable
+            name="drive_module_right_4_link"
+            mass="${drive_module_right_mass}"
+            mass_center="${drive_module_right_mass_center_xyz}"
+            origin_xyz="${drive_module_right_4_origin}"
+            origin_rpy="${drive_module_right_rpy}"
+            mesh_filename="package://rover_description/meshes/MirrorDrive Module_steerable.STL"
+        />
         <joint name="wheel_4_joint" type="continuous">
-            <origin xyz="${wheel_left_4_offset}" rpy="${wheel_right_rpy}"/>
+            <origin xyz="${wheel_right_4_offset}" rpy="${wheel_right_rpy}"/>
             <parent link="drive_module_right_3_link"/>
             <child link="bogie_4_wheel"/>
@@ -126,5 +96,5 @@
         <wheel prefix="bogie_4" />
         <joint name="wheel_5_joint" type="continuous">
-            <origin xyz="${wheel_left_5_offset}" rpy="${wheel_right_rpy}"/>
+            <origin xyz="${wheel_right_5_offset}" rpy="${wheel_right_rpy}"/>
             <parent link="bogie_pivot_right_link"/>
             <child link="bogie_5_wheel"/>
@@ -133,5 +103,5 @@
         <wheel prefix="bogie_5" />
         <joint name="wheel_6_joint" type="continuous">
-            <origin xyz="${wheel_left_6_offset}" rpy="${wheel_right_rpy}"/>
+            <origin xyz="${wheel_right_6_offset}" rpy="${wheel_right_rpy}"/>
             <parent link="drive_module_right_4_link"/>
             <child link="bogie_6_wheel"/>

Commit message: Physics and controll created

File: robot_ws/src/rover_description/urdf/iteso_rover.xacro (robot description, xacro)
@@ -13,4 +13,6 @@
     <!-- Module Steerable -->
     <xacro:include filename="$(find rover_description)/urdf/drive_module_steerable.xacro"/>
+    <!-- Gazebo aspects of the robot -->
+    <xacro:include filename="$(find rover_description)/urdf/iteso_rover.xml"/>
     <!-- Macros calls -->
     <chassis />

File: robot_ws/src/rover_description/urdf/suspension_left.xacro (robot description, xacro)
@@ -31,10 +31,10 @@
             </collision>
         </link>
-        <joint name="rocker_bogie_left" type="continuous">
+        <joint name="rocker_bogie_left_joint" type="continuous">
             <origin xyz="${bogie_pivot_left_offset}" rpy="0.0 0.0 0.0"/>
             <parent link="rocker_left_link"/>
             <child link="bogie_pivot_left_link"/>
             <axis xyz="1.0 0.0 0.0"/>
-            <dynamics damping="0.0" friction="0.0"/>>
+            <dynamics damping="0.0" friction="0.1"/>>
         </joint>
         <link name="bogie_pivot_left_link">
@@ -61,10 +61,20 @@
             </collision>
         </link>
-        <joint name="bogie_drive_left_1" type="continuous">
+        <transmission name="rocker_bogie_left_trans">
+            <type>transmission_interface/SimpleTransmission</type>
+            <joint name="rocker_bogie_left_joint">
+                <hardwareInterface>hardware_interface/EffortJointInterface</hardwareInterface>
+            </joint>
+            <actuator name="rocker_bogie_left_motor">
+                <hardwareInterface>hardware_interface/EffortJointInterface</hardwareInterface>
+                <mechanicalReduction>1</mechanicalReduction>
+            </actuator>
+        </transmission>
+        <joint name="bogie_drive_1_joint" type="continuous">
             <origin xyz="${drive_module_left_1_offset}" rpy="0.0 0.0 0.0"/>
             <parent link="rocker_left_link"/>
             <child link="drive_module_left_1_link"/>
             <axis xyz="0.0 0.0 1.0"/>
-            <dynamics damping="0.0" friction="0.0"/>
+            <dynamics damping="0.0" friction="0.1"/>
         </joint>
         <module_steerable
@@ -76,5 +86,15 @@
             mesh_filename="package://rover_description/meshes/Drive Module_steerable.STL"
         />
-        <joint name="bogie_drive_left_2" type="continuous">
+        <transmission name="bogie_drive_1_trans">
+            <type>transmission_interface/SimpleTransmission</type>
+            <joint name="bogie_drive_1_joint">
+                <hardwareInterface>hardware_interface/EffortJointInterface</hardwareInterface>
+            </joint>
+            <actuator name="bogie_drive_1_motor">
+                <hardwareInterface>hardware_interface/EffortJointInterface</hardwareInterface>
+                <mechanicalReduction>1</mechanicalReduction>
+            </actuator>
+        </transmission>
+        <joint name="bogie_drive_2_joint" type="continuous">
             <origin xyz="${drive_module_left_2_offset}" rpy="0.0 0.0 0.0"/>
             <parent link="bogie_pivot_left_link"/>
@@ -90,4 +110,14 @@
             mesh_filename="package://rover_description/meshes/Drive Module_steerable.STL"
         />
+        <transmission name="bogie_drive_2_trans">
+            <type>transmission_interface/SimpleTransmission</type>
+            <joint name="bogie_drive_2_joint">
+                <hardwareInterface>hardware_interface/EffortJointInterface</hardwareInterface>
+            </joint>
+            <actuator name="bogie_drive_2_motor">
+                <hardwareInterface>hardware_interface/EffortJointInterface</hardwareInterface>
+                <mechanicalReduction>1</mechanicalReduction>
+            </actuator>
+        </transmission>
         <joint name="wheel_1_joint" type="continuous">
             <origin xyz="${wheel_left_1_offset}" rpy="${wheel_left_rpy}"/>
@@ -95,7 +125,17 @@
             <child link="bogie_1_wheel"/>
             <axis xyz="1.0 0.0 0.0"/>
-            <dynamics damping="0.5" friction="0.01"/>
+            <dynamics damping="0.0" friction="0.1"/>
         </joint>
         <wheel prefix="bogie_1" />
+        <transmission name="wheel_1_trans">
+            <type>transmission_interface/SimpleTransmission</type>
+            <joint name="wheel_1_joint">
+                <hardwareInterface>hardware_interface/EffortJointInterface</hardwareInterface>
+            </joint>
+            <actuator name="wheel_1_motor">
+                <hardwareInterface>hardware_interface/EffortJointInterface</hardwareInterface>
+                <mechanicalReduction>1</mechanicalReduction>
+            </actuator>
+        </transmission>
         <joint name="wheel_2_joint" type="continuous">
             <origin xyz="${wheel_left_2_offset}" rpy="${wheel_left_rpy}"/>
@@ -103,7 +143,17 @@
             <child link="bogie_2_wheel"/>
             <axis xyz="1.0 0.0 0.0"/>
-            <dynamics damping="0.5" friction="0.01"/>
+            <dynamics damping="0.0" friction="0.1"/>
         </joint>
         <wheel prefix="bogie_2" />
+        <transmission name="wheel_2_trans">
+            <type>transmission_interface/SimpleTransmission</type>
+            <joint name="wheel_2_joint">
+                <hardwareInterface>hardware_interface/EffortJointInterface</hardwareInterface>
+            </joint>
+            <actuator name="wheel_2_motor">
+                <hardwareInterface>hardware_interface/EffortJointInterface</hardwareInterface>
+                <mechanicalReduction>1</mechanicalReduction>
+            </actuator>
+        </transmission>
         <joint name="wheel_3_joint" type="continuous">
             <origin xyz="${wheel_left_3_offset}" rpy="${wheel_left_rpy}"/>
@@ -111,7 +161,17 @@
             <child link="bogie_3_wheel"/>
             <axis xyz="1.0 0.0 0.0"/>
-            <dynamics damping="0.5" friction="0.01"/>
+            <dynamics damping="0.0" friction="0.1"/>
         </joint>
         <wheel prefix="bogie_3" />
+        <transmission name="wheel_3_trans">
+            <type>transmission_interface/SimpleTransmission</type>
+            <joint name="wheel_3_joint">
+                <hardwareInterface>hardware_interface/EffortJointInterface</hardwareInterface>
+            </joint>
+            <actuator name="wheel_3_motor">
+                <hardwareInterface>hardware_interface/EffortJointInterface</hardwareInterface>
+                <mechanicalReduction>1</mechanicalReduction>
+            </actuator>
+        </transmission>
     </xacro:macro>
 </robot>

File: robot_ws/src/rover_description/urdf/suspension_right.xacro (robot description, xacro)
@@ -31,10 +31,10 @@
             </collision>
         </link>
-        <joint name="rocker_bogie_right" type="continuous">
+        <joint name="rocker_bogie_right_joint" type="continuous">
             <origin xyz="${bogie_pivot_right_offset}" rpy="0.0 0.0 0.0"/>
             <parent link="rocker_right_link"/>
             <child link="bogie_pivot_right_link"/>
             <axis xyz="1.0 0.0 0.0"/>
-            <dynamics damping="0.0" friction="0.0"/>
+            <dynamics damping="0.0" friction="0.1"/>
         </joint>
         <link name="bogie_pivot_right_link">
@@ -61,10 +61,20 @@
             </collision>
         </link>
-        <joint name="bogie_drive_right_3" type="continuous">
+        <transmission name="rocker_bogie_right_trans">
+            <type>transmission_interface/SimpleTransmission</type>
+            <joint name="rocker_bogie_right_joint">
+                <hardwareInterface>hardware_interface/EffortJointInterface</hardwareInterface>
+            </joint>
+            <actuator name="rocker_bogie_right_motor">
+                <hardwareInterface>hardware_interface/EffortJointInterface</hardwareInterface>
+                <mechanicalReduction>1</mechanicalReduction>
+            </actuator>
+        </transmission>
+        <joint name="bogie_drive_3_joint" type="continuous">
             <origin xyz="${drive_module_right_3_offset}" rpy="0.0 0.0 0.0"/>
             <parent link="rocker_right_link"/>
             <child link="drive_module_right_3_link"/>
             <axis xyz="0.0 0.0 1.0"/>
-            <dynamics damping="0.0" friction="0.0"/>
+            <dynamics damping="0.0" friction="0.1"/>
         </joint>
         <module_steerable
@@ -76,10 +86,20 @@
             mesh_filename="package://rover_description/meshes/MirrorDrive Module_steerable.STL"
         />
-        <joint name="bogie_drive_right_4" type="continuous">
+        <transmission name="bogie_drive_3_trans">
+            <type>transmission_interface/SimpleTransmission</type>
+            <joint name="bogie_drive_3_joint">
+                <hardwareInterface>hardware_interface/EffortJointInterface</hardwareInterface>
+            </joint>
+            <actuator name="bogie_drive_3_motor">
+                <hardwareInterface>hardware_interface/EffortJointInterface</hardwareInterface>
+                <mechanicalReduction>1</mechanicalReduction>
+            </actuator>
+        </transmission>
+        <joint name="bogie_drive_4_joint" type="continuous">
             <origin xyz="${drive_module_right_4_offset}" rpy="0.0 0.0 0.0"/>
             <parent link="bogie_pivot_right_link"/>
             <child link="drive_module_right_4_link"/>
             <axis xyz="0.0 0.0 1.0"/>
-            <dynamics damping="0.0" friction="0.0"/>
+            <dynamics damping="0.0" friction="0.1"/>
         </joint>
         <module_steerable
@@ -91,4 +111,14 @@
             mesh_filename="package://rover_description/meshes/MirrorDrive Module_steerable.STL"
         />
+        <transmission name="bogie_drive_4_trans">
+            <type>transmission_interface/SimpleTransmission</type>
+            <joint name="bogie_drive_4_joint">
+                <hardwareInterface>hardware_interface/EffortJointInterface</hardwareInterface>
+            </joint>
+            <actuator name="bogie_drive_4_motor">
+                <hardwareInterface>hardware_interface/EffortJointInterface</hardwareInterface>
+                <mechanicalReduction>1</mechanicalReduction>
+            </actuator>
+        </transmission>
         <joint name="wheel_4_joint" type="continuous">
             <origin xyz="${wheel_right_4_offset}" rpy="${wheel_right_rpy}"/>
@@ -96,7 +126,17 @@
             <child link="bogie_4_wheel"/>
             <axis xyz="1.0 0.0 0.0"/>
-            <dynamics damping="0.5" friction="0.01"/>
+            <dynamics damping="0.0" friction="0.00"/>
         </joint>
         <wheel prefix="bogie_4" />
+        <transmission name="wheel_4_trans">
+            <type>transmission_interface/SimpleTransmission</type>
+            <joint name="wheel_4_joint">
+                <hardwareInterface>hardware_interface/EffortJointInterface</hardwareInterface>
+            </joint>
+            <actuator name="wheel_4_motor">
+                <hardwareInterface>hardware_interface/EffortJointInterface</hardwareInterface>
+                <mechanicalReduction>1</mechanicalReduction>
+            </actuator>
+        </transmission>
         <joint name="wheel_5_joint" type="continuous">
             <origin xyz="${wheel_right_5_offset}" rpy="${wheel_right_rpy}"/>
@@ -104,7 +144,17 @@
             <child link="bogie_5_wheel"/>
             <axis xyz="1.0 0.0 0.0"/>
-            <dynamics damping="0.5" friction="0.01"/>
+            <dynamics damping="0.0" friction="0.1"/>
         </joint>
         <wheel prefix="bogie_5" />
+        <transmission name="wheel_5_trans">
+            <type>transmission_interface/SimpleTransmission</type>
+            <joint name="wheel_5_joint">
+                <hardwareInterface>hardware_interface/EffortJointInterface</hardwareInterface>
+            </joint>
+            <actuator name="wheel_5_motor">
+                <hardwareInterface>hardware_interface/EffortJointInterface</hardwareInterface>
+                <mechanicalReduction>1</mechanicalReduction>
+            </actuator>
+        </transmission>
         <joint name="wheel_6_joint" type="continuous">
             <origin xyz="${wheel_right_6_offset}" rpy="${wheel_right_rpy}"/>
@@ -112,7 +162,17 @@
             <child link="bogie_6_wheel"/>
             <axis xyz="1.0 0.0 0.0"/>
-            <dynamics damping="0.5" friction="0.01"/>
+            <dynamics damping="0.0" friction="0.1"/>
         </joint>
         <wheel prefix="bogie_6" />
+        <transmission name="wheel_6_trans">
+            <type>transmission_interface/SimpleTransmission</type>
+            <joint name="wheel_6_joint">
+                <hardwareInterface>hardware_interface/EffortJointInterface</hardwareInterface>
+            </joint>
+            <actuator name="wheel_6_motor">
+                <hardwareInterface>hardware_interface/EffortJointInterface</hardwareInterface>
+                <mechanicalReduction>1</mechanicalReduction>
+            </actuator>
+        </transmission>
     </xacro:macro>
 </robot>
