Commit message: Physiscs issues

File: simulation_ws/src/rover_description/urdf/chassis.xacro (robot description, xacro)
@@ -13,7 +13,10 @@
                 <origin xyz="${chassis_mass_center_xyz}" rpy="0.0 0.0 0.0"/>
                 <mass value="${chassis_mass}"/>
-                <inertia    ixx="0.0860"    ixy="-0.0008"   ixz="-0.0003"
-                                            iyy="0.0483"    iyz="-0.0099"
-                                                            izz="0.0994"/>
+                <inertia    ixx="${chassis_mass * 0.0860}"
+                            ixy="${chassis_mass * -0.0008}"
+                            ixz="${chassis_mass * -0.0003}"
+                            iyy="${chassis_mass * 0.0483}"
+                            iyz="${chassis_mass * -0.0099}"
+                            izz="${chassis_mass * 0.0994}"/>
             </inertial>
             <visual>

File: simulation_ws/src/rover_description/urdf/drive_module_steerable.xacro (robot description, xacro)
@@ -6,7 +6,10 @@
                 <origin xyz="${mass_center}" rpy="${origin_rpy}"/>
                 <mass value="${mass}"/>
-                <inertia    ixx="0.0102"    ixy="0.0001"    ixz="0.0"
-                                            iyy="0.0063"    iyz="-0.0018"
-                                                            izz="0.0049"/>
+                <inertia    ixx="${mass * 0.0107}"
+                            ixy="${mass * 0.0003}"
+                            ixz="${mass * -0.0003}"
+                            iyy="${mass * 0.0070}"
+                            iyz="${mass * -0.0020}"
+                            izz="${mass * 0.0054}"/>
             </inertial>
             <visual name="">

File: simulation_ws/src/rover_description/urdf/iteso_rover.xacro (robot description, xacro)
@@ -13,9 +13,9 @@
     <!-- Module Steerable -->
     <xacro:include filename="$(find rover_description)/urdf/drive_module_steerable.xacro"/>
-    <!-- Gazebo aspects of the robot -->
-    <xacro:include filename="$(find rover_description)/urdf/iteso_rover.xml"/>
     <!-- Macros calls -->
     <chassis />
     <suspension_left />
     <suspension_right />
+    <!-- Gazebo aspects of the robot -->
+    <xacro:include filename="$(find rover_description)/urdf/iteso_rover.xml"/>
 </robot>

File: simulation_ws/src/rover_description/urdf/suspension_left.xacro (robot description, xacro)
@@ -12,7 +12,10 @@
                 <origin xyz="${rocker_left_mass_center_xyz}" rpy="0.0 0.0 0.0"/>
                 <mass value="${rocker_left_mass}"/>
-                <inertia    ixx="0.0077"    ixy="-0.0012"   ixz="0.0"
-                                            iyy="0.0006"    iyz="-0.0002"
-                                                            izz="0.0078"/>
+                <inertia    ixx="${rocker_left_mass * 0.0093}"
+                            ixy="${rocker_left_mass * -0.0022}"
+                            ixz="${rocker_left_mass * -0.0005}"
+                            iyy="${rocker_left_mass * 0.0015}"
+                            iyz="${rocker_left_mass * 0.0003}"
+                            izz="${rocker_left_mass * 0.0098}"/>
             </inertial>
             <visual>
@@ -36,5 +39,6 @@
             <child link="bogie_pivot_left_link"/>
             <axis xyz="1.0 0.0 0.0"/>
-            <dynamics damping="0.0" friction="0.1"/>>
+            <dynamics damping="0.1" friction="0.05"/>
+            <limit effort="100" velocity="100" />
         </joint>
         <link name="bogie_pivot_left_link">
@@ -42,7 +46,10 @@
                 <origin xyz="${bogie_pivot_left_mass_center_xyz}" rpy="0.0 0.0 0.0"/>
                 <mass value="${bogie_pivot_left_mass}"/>
-                <inertia    ixx="0.0059"    ixy="-0.0002"    ixz="0.0002"
-                                            iyy="0.0014"    iyz="0.002"
-                                                            izz="0.0051"/>
+                <inertia    ixx="${bogie_pivot_left_mass * 0.0061}"
+                            ixy="${bogie_pivot_left_mass * 0.0}"
+                            ixz="${bogie_pivot_left_mass * -0.0006}"
+                            iyy="${bogie_pivot_left_mass * 0.0024}"
+                            iyz="${bogie_pivot_left_mass * 0.002}"
+                            izz="${bogie_pivot_left_mass * 0.006}"/>
             </inertial>
             <visual>
@@ -76,5 +83,6 @@
             <child link="drive_module_left_1_link"/>
             <axis xyz="0.0 0.0 1.0"/>
-            <dynamics damping="0.0" friction="0.1"/>
+            <dynamics damping="0.1" friction="0.05"/>
+            <limit effort="100" velocity="100" />
         </joint>
         <module_steerable
@@ -101,4 +109,6 @@
             <child link="drive_module_left_2_link"/>
             <axis xyz="0.0 0.0 1.0"/>
+            <dynamics damping="0.1" friction="0.05"/>
+            <limit effort="100" velocity="100" />
         </joint>
         <module_steerable
@@ -125,5 +135,6 @@
             <child link="bogie_1_wheel"/>
             <axis xyz="1.0 0.0 0.0"/>
-            <dynamics damping="0.0" friction="0.1"/>
+            <dynamics damping="0.1" friction="0.05"/>
+            <limit effort="100" velocity="100" />
         </joint>
         <wheel prefix="bogie_1" />
@@ -143,5 +154,6 @@
             <child link="bogie_2_wheel"/>
             <axis xyz="1.0 0.0 0.0"/>
-            <dynamics damping="0.0" friction="0.1"/>
+            <dynamics damping="0.1" friction="0.05"/>
+            <limit effort="100" velocity="100" />
         </joint>
         <wheel prefix="bogie_2" />
@@ -161,5 +173,6 @@
             <child link="bogie_3_wheel"/>
             <axis xyz="1.0 0.0 0.0"/>
-            <dynamics damping="0.0" friction="0.1"/>
+            <dynamics damping="0.1" friction="0.05"/>
+            <limit effort="100" velocity="100" />
         </joint>
         <wheel prefix="bogie_3" />

File: simulation_ws/src/rover_description/urdf/suspension_right.xacro (robot description, xacro)
@@ -12,7 +12,10 @@
                 <origin xyz="${rocker_right_mass_center_xyz}" rpy="0.0 0.0 0.0"/>
                 <mass value="${rocker_right_mass}"/>
-                <inertia    ixx="0.0077"    ixy="-0.0005"   ixz="0.0022"
-                                            iyy="0.0098"    iyz="-0.0003"
-                                                            izz="0.0015"/>
+                <inertia    ixx="${rocker_right_mass * 0.0206}"
+                            ixy="${rocker_right_mass * 0.0047}"
+                            ixz="${rocker_right_mass * -0.0030}"
+                            iyy="${rocker_right_mass * 0.0356}"
+                            iyz="${rocker_right_mass * 0.0001}"
+                            izz="${rocker_right_mass * 0.0306}"/>
             </inertial>
             <visual>
@@ -36,5 +39,6 @@
             <child link="bogie_pivot_right_link"/>
             <axis xyz="1.0 0.0 0.0"/>
-            <dynamics damping="0.0" friction="0.1"/>
+            <dynamics damping="0.1" friction="0.05"/>
+            <limit effort="100" velocity="100" />
         </joint>
         <link name="bogie_pivot_right_link">
@@ -42,7 +46,10 @@
                 <origin xyz="${bogie_pivot_right_mass_center_xyz}" rpy="0.0 0.0 0.0"/>
                 <mass value="${bogie_pivot_right_mass}"/>
-                <inertia    ixx="0.0684"    ixy="0.0038"    ixz="0.0"
-                                            iyy="0.0572"    iyz="-0.0028"
-                                                            izz="0.0425"/>
+                <inertia    ixx="${bogie_pivot_right_mass * 0.0024}"
+                            ixy="${bogie_pivot_right_mass * 0.0}"
+                            ixz="${bogie_pivot_right_mass * -0.002}"
+                            iyy="${bogie_pivot_right_mass * 0.0061}"
+                            iyz="${bogie_pivot_right_mass * -0.0006}"
+                            izz="${bogie_pivot_right_mass * 0.006}"/>
             </inertial>
             <visual>
@@ -76,5 +83,6 @@
             <child link="drive_module_right_3_link"/>
             <axis xyz="0.0 0.0 1.0"/>
-            <dynamics damping="0.0" friction="0.1"/>
+            <dynamics damping="0.1" friction="0.05"/>
+            <limit effort="100" velocity="100" />
         </joint>
         <module_steerable
@@ -82,5 +90,5 @@
             mass="${drive_module_right_mass}"
             mass_center="${drive_module_right_mass_center_xyz}"
-            origin_xyz="${drive_module_right_4_origin}"
+            origin_xyz="${drive_module_right_3_origin}"
             origin_rpy="${drive_module_right_rpy}"
             mesh_filename="package://rover_description/meshes/MirrorDrive Module_steerable.STL"
@@ -101,5 +109,6 @@
             <child link="drive_module_right_4_link"/>
             <axis xyz="0.0 0.0 1.0"/>
-            <dynamics damping="0.0" friction="0.1"/>
+            <dynamics damping="0.1" friction="0.05"/>
+            <limit effort="100" velocity="100" />
         </joint>
         <module_steerable
@@ -126,5 +135,6 @@
             <child link="bogie_4_wheel"/>
             <axis xyz="1.0 0.0 0.0"/>
-            <dynamics damping="0.0" friction="0.00"/>
+            <dynamics damping="0.1" friction="0.05"/>
+            <limit effort="100" velocity="100" />
         </joint>
         <wheel prefix="bogie_4" />
@@ -144,5 +154,6 @@
             <child link="bogie_5_wheel"/>
             <axis xyz="1.0 0.0 0.0"/>
-            <dynamics damping="0.0" friction="0.1"/>
+            <dynamics damping="0.1" friction="0.05"/>
+            <limit effort="100" velocity="100" />
         </joint>
         <wheel prefix="bogie_5" />
@@ -162,5 +173,6 @@
             <child link="bogie_6_wheel"/>
             <axis xyz="1.0 0.0 0.0"/>
-            <dynamics damping="0.0" friction="0.1"/>
+            <dynamics damping="0.1" friction="0.05"/>
+            <limit effort="100" velocity="100" />
         </joint>
         <wheel prefix="bogie_6" />

File: simulation_ws/src/rover_description/urdf/wheel.xacro (robot description, xacro)
@@ -6,7 +6,10 @@
                 <origin xyz="${wheel_mass_center_xyz}" rpy="0.0 0.0 0.0"/>
                 <mass value="${wheel_mass}"/>
-                <inertia ixx="0.0004"   ixy="0.0"       ixz="0.0"
-                                        iyy="0.0002"    iyz="-0.0001"
-                                                        izz="0.0003"/>
+                <inertia    ixx="${wheel_mass * 0.00032225}"
+                            ixy="${wheel_mass * 0.0}"
+                            ixz="${wheel_mass * -0.00000081}"
+                            iyy="${wheel_mass * 0.00025631}"
+                            iyz="${wheel_mass * 0.0}"
+                            izz="${wheel_mass * 0.00025631}"/>
             </inertial>
             <visual>

Commit message: Testing control

File: simulation_ws/src/rover_description/urdf/chassis.xacro (robot description, xacro)
@@ -13,10 +13,10 @@
                 <origin xyz="${chassis_mass_center_xyz}" rpy="0.0 0.0 0.0"/>
                 <mass value="${chassis_mass}"/>
-                <inertia    ixx="${chassis_mass * 0.0860}"
-                            ixy="${chassis_mass * -0.0008}"
-                            ixz="${chassis_mass * -0.0003}"
-                            iyy="${chassis_mass * 0.0483}"
-                            iyz="${chassis_mass * -0.0099}"
-                            izz="${chassis_mass * 0.0994}"/>
+                <inertia    ixx="${ 0.0860}"
+                            ixy="${ -0.0008}"
+                            ixz="${ -0.0003}"
+                            iyy="${ 0.0483}"
+                            iyz="${ -0.0099}"
+                            izz="${ 0.0994}"/>
             </inertial>
             <visual>

File: simulation_ws/src/rover_description/urdf/drive_module_steerable.xacro (robot description, xacro)
@@ -6,10 +6,10 @@
                 <origin xyz="${mass_center}" rpy="${origin_rpy}"/>
                 <mass value="${mass}"/>
-                <inertia    ixx="${mass * 0.0107}"
-                            ixy="${mass * 0.0003}"
-                            ixz="${mass * -0.0003}"
-                            iyy="${mass * 0.0070}"
-                            iyz="${mass * -0.0020}"
-                            izz="${mass * 0.0054}"/>
+                <inertia    ixx="${ 0.0107}"
+                            ixy="${ 0.0003}"
+                            ixz="${ -0.0003}"
+                            iyy="${ 0.0070}"
+                            iyz="${ -0.0020}"
+                            izz="${ 0.0054}"/>
             </inertial>
             <visual name="">

File: simulation_ws/src/rover_description/urdf/suspension_left.xacro (robot description, xacro)
@@ -12,10 +12,10 @@
                 <origin xyz="${rocker_left_mass_center_xyz}" rpy="0.0 0.0 0.0"/>
                 <mass value="${rocker_left_mass}"/>
-                <inertia    ixx="${rocker_left_mass * 0.0093}"
-                            ixy="${rocker_left_mass * -0.0022}"
-                            ixz="${rocker_left_mass * -0.0005}"
-                            iyy="${rocker_left_mass * 0.0015}"
-                            iyz="${rocker_left_mass * 0.0003}"
-                            izz="${rocker_left_mass * 0.0098}"/>
+                <inertia    ixx="${ 0.0093}"
+                            ixy="${ -0.0022}"
+                            ixz="${ -0.0005}"
+                            iyy="${ 0.0015}"
+                            iyz="${ 0.0003}"
+                            izz="${ 0.0098}"/>
             </inertial>
             <visual>
@@ -39,5 +39,5 @@
             <child link="bogie_pivot_left_link"/>
             <axis xyz="1.0 0.0 0.0"/>
-            <dynamics damping="0.01" friction="0.0"/>
+            <dynamics damping="0.0" friction="0.0"/>
             <limit effort="30" velocity="100" />
         </joint>
@@ -46,10 +46,10 @@
                 <origin xyz="${bogie_pivot_left_mass_center_xyz}" rpy="0.0 0.0 0.0"/>
                 <mass value="${bogie_pivot_left_mass}"/>
-                <inertia    ixx="${bogie_pivot_left_mass * 0.0061}"
-                            ixy="${bogie_pivot_left_mass * 0.0}"
-                            ixz="${bogie_pivot_left_mass * -0.0006}"
-                            iyy="${bogie_pivot_left_mass * 0.0024}"
-                            iyz="${bogie_pivot_left_mass * 0.002}"
-                            izz="${bogie_pivot_left_mass * 0.006}"/>
+                <inertia    ixx="${ 0.0061}"
+                            ixy="${ 0.0}"
+                            ixz="${ -0.0006}"
+                            iyy="${ 0.0024}"
+                            iyz="${ 0.002}"
+                            izz="${ 0.006}"/>
             </inertial>
             <visual>
@@ -83,5 +83,5 @@
             <child link="drive_module_left_1_link"/>
             <axis xyz="0.0 0.0 1.0"/>
-            <dynamics damping="0.01" friction="0.0"/>
+            <dynamics damping="0.0" friction="0.0"/>
             <limit effort="30" velocity="100" />
         </joint>
@@ -109,5 +109,5 @@
             <child link="drive_module_left_2_link"/>
             <axis xyz="0.0 0.0 1.0"/>
-            <dynamics damping="0.01" friction="0.0"/>
+            <dynamics damping="0.0" friction="0.0"/>
             <limit effort="30" velocity="100" />
         </joint>
@@ -135,5 +135,5 @@
             <child link="bogie_1_wheel"/>
             <axis xyz="1.0 0.0 0.0"/>
-            <dynamics damping="0.01" friction="0.1"/>
+            <dynamics damping="0.0" friction="0.5"/>
             <limit effort="30" velocity="100" />
         </joint>
@@ -154,5 +154,5 @@
             <child link="bogie_2_wheel"/>
             <axis xyz="1.0 0.0 0.0"/>
-            <dynamics damping="0.01" friction="0.1"/>
+            <dynamics damping="0.0" friction="0.5"/>
             <limit effort="30" velocity="100" />
         </joint>
@@ -173,5 +173,5 @@
             <child link="bogie_3_wheel"/>
             <axis xyz="1.0 0.0 0.0"/>
-            <dynamics damping="0.01" friction="0.1"/>
+            <dynamics damping="0.0" friction="0.5"/>
             <limit effort="30" velocity="100" />
         </joint>

File: simulation_ws/src/rover_description/urdf/suspension_right.xacro (robot description, xacro)
@@ -12,10 +12,10 @@
                 <origin xyz="${rocker_right_mass_center_xyz}" rpy="0.0 0.0 0.0"/>
                 <mass value="${rocker_right_mass}"/>
-                <inertia    ixx="${rocker_right_mass * 0.0206}"
-                            ixy="${rocker_right_mass * 0.0047}"
-                            ixz="${rocker_right_mass * -0.0030}"
-                            iyy="${rocker_right_mass * 0.0356}"
-                            iyz="${rocker_right_mass * 0.0001}"
-                            izz="${rocker_right_mass * 0.0306}"/>
+                <inertia    ixx="${ 0.0206}"
+                            ixy="${ 0.0047}"
+                            ixz="${ -0.0030}"
+                            iyy="${ 0.0356}"
+                            iyz="${ 0.0001}"
+                            izz="${ 0.0306}"/>
             </inertial>
             <visual>
@@ -39,5 +39,5 @@
             <child link="bogie_pivot_right_link"/>
             <axis xyz="1.0 0.0 0.0"/>
-            <dynamics damping="0.01" friction="0.0"/>
+            <dynamics  damping="0.0" friction="0.0"/>
             <limit effort="30" velocity="100" />
         </joint>
@@ -46,10 +46,10 @@
                 <origin xyz="${bogie_pivot_right_mass_center_xyz}" rpy="0.0 0.0 0.0"/>
                 <mass value="${bogie_pivot_right_mass}"/>
-                <inertia    ixx="${bogie_pivot_right_mass * 0.0024}"
-                            ixy="${bogie_pivot_right_mass * 0.0}"
-                            ixz="${bogie_pivot_right_mass * -0.002}"
-                            iyy="${bogie_pivot_right_mass * 0.0061}"
-                            iyz="${bogie_pivot_right_mass * -0.0006}"
-                            izz="${bogie_pivot_right_mass * 0.006}"/>
+                <inertia    ixx="${ 0.0024}"
+                            ixy="${ 0.0}"
+                            ixz="${ -0.002}"
+                            iyy="${ 0.0061}"
+                            iyz="${ -0.0006}"
+                            izz="${ 0.006}"/>
             </inertial>
             <visual>
@@ -83,5 +83,5 @@
             <child link="drive_module_right_3_link"/>
             <axis xyz="0.0 0.0 1.0"/>
-            <dynamics damping="0.01" friction="0.0"/>
+            <dynamics  damping="0.0" friction="0.0"/>
             <limit effort="30" velocity="100" />
         </joint>
@@ -109,5 +109,5 @@
             <child link="drive_module_right_4_link"/>
             <axis xyz="0.0 0.0 1.0"/>
-            <dynamics damping="0.01" friction="0.0"/>
+            <dynamics  damping="0.0" friction="0.0"/>
             <limit effort="30" velocity="100" />
         </joint>
@@ -135,5 +135,5 @@
             <child link="bogie_4_wheel"/>
             <axis xyz="1.0 0.0 0.0"/>
-            <dynamics damping="0.01" friction="0.1"/>
+            <dynamics  damping="0.0" friction="0.5"/>
             <limit effort="30" velocity="100" />
         </joint>
@@ -154,5 +154,5 @@
             <child link="bogie_5_wheel"/>
             <axis xyz="1.0 0.0 0.0"/>
-            <dynamics damping="0.01" friction="0.1"/>
+            <dynamics  damping="0.0" friction="0.5"/>
             <limit effort="30" velocity="100" />
         </joint>
@@ -173,5 +173,5 @@
             <child link="bogie_6_wheel"/>
             <axis xyz="1.0 0.0 0.0"/>
-            <dynamics damping="0.01" friction="0.1"/>
+            <dynamics  damping="0.0" friction="0.5"/>
             <limit effort="30" velocity="100" />
         </joint>

File: simulation_ws/src/rover_description/urdf/wheel.xacro (robot description, xacro)
@@ -6,10 +6,10 @@
                 <origin xyz="${wheel_mass_center_xyz}" rpy="0.0 0.0 0.0"/>
                 <mass value="${wheel_mass}"/>
-                <inertia    ixx="${wheel_mass * 0.00032225}"
-                            ixy="${wheel_mass * 0.0}"
-                            ixz="${wheel_mass * -0.00000081}"
-                            iyy="${wheel_mass * 0.00025631}"
-                            iyz="${wheel_mass * 0.0}"
-                            izz="${wheel_mass * 0.00025631}"/>
+                <inertia    ixx="${ 0.00032225}"
+                            ixy="${ 0.0}"
+                            ixz="${ -0.00000081}"
+                            iyy="${ 0.00025631}"
+                            iyz="${ 0.0}"
+                            izz="${ 0.00025631}"/>
             </inertial>
             <visual>
