Commit message: Test for AWS robomaker

File: simulation_ws/src/rover_description/urdf/suspension_left.xacro (robot description, xacro)
@@ -39,6 +39,6 @@
             <child link="bogie_pivot_left_link"/>
             <axis xyz="1.0 0.0 0.0"/>
-            <dynamics damping="0.1" friction="0.05"/>
-            <limit effort="100" velocity="100" />
+            <dynamics damping="0.01" friction="0.0"/>
+            <limit effort="30" velocity="100" />
         </joint>
         <link name="bogie_pivot_left_link">
@@ -83,6 +83,6 @@
             <child link="drive_module_left_1_link"/>
             <axis xyz="0.0 0.0 1.0"/>
-            <dynamics damping="0.1" friction="0.05"/>
-            <limit effort="100" velocity="100" />
+            <dynamics damping="0.01" friction="0.0"/>
+            <limit effort="30" velocity="100" />
         </joint>
         <module_steerable
@@ -109,6 +109,6 @@
             <child link="drive_module_left_2_link"/>
             <axis xyz="0.0 0.0 1.0"/>
-            <dynamics damping="0.1" friction="0.05"/>
-            <limit effort="100" velocity="100" />
+            <dynamics damping="0.01" friction="0.0"/>
+            <limit effort="30" velocity="100" />
         </joint>
         <module_steerable
@@ -135,6 +135,6 @@
             <child link="bogie_1_wheel"/>
             <axis xyz="1.0 0.0 0.0"/>
-            <dynamics damping="0.1" friction="0.05"/>
-            <limit effort="100" velocity="100" />
+            <dynamics damping="0.01" friction="0.0"/>
+            <limit effort="30" velocity="100" />
         </joint>
         <wheel prefix="bogie_1" />
@@ -154,6 +154,6 @@
             <child link="bogie_2_wheel"/>
             <axis xyz="1.0 0.0 0.0"/>
-            <dynamics damping="0.1" friction="0.05"/>
-            <limit effort="100" velocity="100" />
+            <dynamics damping="0.01" friction="0.0"/>
+            <limit effort="30" velocity="100" />
         </joint>
         <wheel prefix="bogie_2" />
@@ -173,6 +173,6 @@
             <child link="bogie_3_wheel"/>
             <axis xyz="1.0 0.0 0.0"/>
-            <dynamics damping="0.1" friction="0.05"/>
-            <limit effort="100" velocity="100" />
+            <dynamics damping="0.01" friction="0.0"/>
+            <limit effort="30" velocity="100" />
         </joint>
         <wheel prefix="bogie_3" />

File: simulation_ws/src/rover_description/urdf/suspension_right.xacro (robot description, xacro)
@@ -39,6 +39,6 @@
             <child link="bogie_pivot_right_link"/>
             <axis xyz="1.0 0.0 0.0"/>
-            <dynamics damping="0.1" friction="0.05"/>
-            <limit effort="100" velocity="100" />
+            <dynamics damping="0.01" friction="0.0"/>
+            <limit effort="30" velocity="100" />
         </joint>
         <link name="bogie_pivot_right_link">
@@ -83,6 +83,6 @@
             <child link="drive_module_right_3_link"/>
             <axis xyz="0.0 0.0 1.0"/>
-            <dynamics damping="0.1" friction="0.05"/>
-            <limit effort="100" velocity="100" />
+            <dynamics damping="0.01" friction="0.0"/>
+            <limit effort="30" velocity="100" />
         </joint>
         <module_steerable
@@ -109,6 +109,6 @@
             <child link="drive_module_right_4_link"/>
             <axis xyz="0.0 0.0 1.0"/>
-            <dynamics damping="0.1" friction="0.05"/>
-            <limit effort="100" velocity="100" />
+            <dynamics damping="0.01" friction="0.0"/>
+            <limit effort="30" velocity="100" />
         </joint>
         <module_steerable
@@ -135,6 +135,6 @@
             <child link="bogie_4_wheel"/>
             <axis xyz="1.0 0.0 0.0"/>
-            <dynamics damping="0.1" friction="0.05"/>
-            <limit effort="100" velocity="100" />
+            <dynamics damping="0.01" friction="0.0"/>
+            <limit effort="30" velocity="100" />
         </joint>
         <wheel prefix="bogie_4" />
@@ -154,6 +154,6 @@
             <child link="bogie_5_wheel"/>
             <axis xyz="1.0 0.0 0.0"/>
-            <dynamics damping="0.1" friction="0.05"/>
-            <limit effort="100" velocity="100" />
+            <dynamics damping="0.01" friction="0.0"/>
+            <limit effort="30" velocity="100" />
         </joint>
         <wheel prefix="bogie_5" />
@@ -173,6 +173,6 @@
             <child link="bogie_6_wheel"/>
             <axis xyz="1.0 0.0 0.0"/>
-            <dynamics damping="0.1" friction="0.05"/>
-            <limit effort="100" velocity="100" />
+            <dynamics damping="0.01" friction="0.0"/>
+            <limit effort="30" velocity="100" />
         </joint>
         <wheel prefix="bogie_6" />

Commit message: Try AWS rqt and fix PID wheels controllers values

File: simulation_ws/src/rover_description/urdf/suspension_left.xacro (robot description, xacro)
@@ -135,5 +135,5 @@
             <child link="bogie_1_wheel"/>
             <axis xyz="1.0 0.0 0.0"/>
-            <dynamics damping="0.01" friction="0.0"/>
+            <dynamics damping="0.01" friction="0.1"/>
             <limit effort="30" velocity="100" />
         </joint>
@@ -154,5 +154,5 @@
             <child link="bogie_2_wheel"/>
             <axis xyz="1.0 0.0 0.0"/>
-            <dynamics damping="0.01" friction="0.0"/>
+            <dynamics damping="0.01" friction="0.1"/>
             <limit effort="30" velocity="100" />
         </joint>
@@ -173,5 +173,5 @@
             <child link="bogie_3_wheel"/>
             <axis xyz="1.0 0.0 0.0"/>
-            <dynamics damping="0.01" friction="0.0"/>
+            <dynamics damping="0.01" friction="0.1"/>
             <limit effort="30" velocity="100" />
         </joint>

File: simulation_ws/src/rover_description/urdf/suspension_right.xacro (robot description, xacro)
@@ -135,5 +135,5 @@
             <child link="bogie_4_wheel"/>
             <axis xyz="1.0 0.0 0.0"/>
-            <dynamics damping="0.01" friction="0.0"/>
+            <dynamics damping="0.01" friction="0.1"/>
             <limit effort="30" velocity="100" />
         </joint>
@@ -154,5 +154,5 @@
             <child link="bogie_5_wheel"/>
             <axis xyz="1.0 0.0 0.0"/>
-            <dynamics damping="0.01" friction="0.0"/>
+            <dynamics damping="0.01" friction="0.1"/>
             <limit effort="30" velocity="100" />
         </joint>
@@ -173,5 +173,5 @@
             <child link="bogie_6_wheel"/>
             <axis xyz="1.0 0.0 0.0"/>
-            <dynamics damping="0.01" friction="0.0"/>
+            <dynamics damping="0.01" friction="0.1"/>
             <limit effort="30" velocity="100" />
         </joint>

Commit message: robot velocity controllers

File: simulation_ws/src/rover_description/urdf/suspension_left.xacro (robot description, xacro)
@@ -83,5 +83,5 @@
             <child link="drive_module_left_1_link"/>
             <axis xyz="0.0 0.0 1.0"/>
-            <dynamics damping="0.0" friction="0.0"/>
+            <dynamics damping="0.5" friction="0.5"/>
             <limit effort="30" velocity="100" />
         </joint>
@@ -109,5 +109,5 @@
             <child link="drive_module_left_2_link"/>
             <axis xyz="0.0 0.0 1.0"/>
-            <dynamics damping="0.0" friction="0.0"/>
+            <dynamics damping="0.0" friction="0.5"/>
             <limit effort="30" velocity="100" />
         </joint>
@@ -142,8 +142,8 @@
             <type>transmission_interface/SimpleTransmission</type>
             <joint name="wheel_1_joint">
-                <hardwareInterface>hardware_interface/EffortJointInterface</hardwareInterface>
+                <hardwareInterface>hardware_interface/VelocityJointInterface</hardwareInterface>
             </joint>
             <actuator name="wheel_1_motor">
-                <hardwareInterface>hardware_interface/EffortJointInterface</hardwareInterface>
+                <hardwareInterface>hardware_interface/VelocityJointInterface</hardwareInterface>
                 <mechanicalReduction>1</mechanicalReduction>
             </actuator>
@@ -161,8 +161,8 @@
             <type>transmission_interface/SimpleTransmission</type>
             <joint name="wheel_2_joint">
-                <hardwareInterface>hardware_interface/EffortJointInterface</hardwareInterface>
+                <hardwareInterface>hardware_interface/VelocityJointInterface</hardwareInterface>
             </joint>
             <actuator name="wheel_2_motor">
-                <hardwareInterface>hardware_interface/EffortJointInterface</hardwareInterface>
+                <hardwareInterface>hardware_interface/VelocityJointInterface</hardwareInterface>
                 <mechanicalReduction>1</mechanicalReduction>
             </actuator>
@@ -180,8 +180,8 @@
             <type>transmission_interface/SimpleTransmission</type>
             <joint name="wheel_3_joint">
-                <hardwareInterface>hardware_interface/EffortJointInterface</hardwareInterface>
+                <hardwareInterface>hardware_interface/VelocityJointInterface</hardwareInterface>
             </joint>
             <actuator name="wheel_3_motor">
-                <hardwareInterface>hardware_interface/EffortJointInterface</hardwareInterface>
+                <hardwareInterface>hardware_interface/VelocityJointInterface</hardwareInterface>
                 <mechanicalReduction>1</mechanicalReduction>
             </actuator>

File: simulation_ws/src/rover_description/urdf/suspension_right.xacro (robot description, xacro)
@@ -83,5 +83,5 @@
             <child link="drive_module_right_3_link"/>
             <axis xyz="0.0 0.0 1.0"/>
-            <dynamics  damping="0.0" friction="0.0"/>
+            <dynamics  damping="0.0" friction="0.5"/>
             <limit effort="30" velocity="100" />
         </joint>
@@ -109,5 +109,5 @@
             <child link="drive_module_right_4_link"/>
             <axis xyz="0.0 0.0 1.0"/>
-            <dynamics  damping="0.0" friction="0.0"/>
+            <dynamics  damping="0.0" friction="0.5"/>
             <limit effort="30" velocity="100" />
         </joint>
@@ -134,5 +134,5 @@
             <parent link="drive_module_right_3_link"/>
             <child link="bogie_4_wheel"/>
-            <axis xyz="1.0 0.0 0.0"/>
+            <axis xyz="-1.0 0.0 0.0"/>
             <dynamics  damping="0.0" friction="0.5"/>
             <limit effort="30" velocity="100" />
@@ -142,8 +142,8 @@
             <type>transmission_interface/SimpleTransmission</type>
             <joint name="wheel_4_joint">
-                <hardwareInterface>hardware_interface/EffortJointInterface</hardwareInterface>
+                <hardwareInterface>hardware_interface/VelocityJointInterface</hardwareInterface>
             </joint>
             <actuator name="wheel_4_motor">
-                <hardwareInterface>hardware_interface/EffortJointInterface</hardwareInterface>
+                <hardwareInterface>hardware_interface/VelocityJointInterface</hardwareInterface>
                 <mechanicalReduction>1</mechanicalReduction>
             </actuator>
@@ -153,5 +153,5 @@
             <parent link="bogie_pivot_right_link"/>
             <child link="bogie_5_wheel"/>
-            <axis xyz="1.0 0.0 0.0"/>
+            <axis xyz="-1.0 0.0 0.0"/>
             <dynamics  damping="0.0" friction="0.5"/>
             <limit effort="30" velocity="100" />
@@ -161,8 +161,8 @@
             <type>transmission_interface/SimpleTransmission</type>
             <joint name="wheel_5_joint">
-                <hardwareInterface>hardware_interface/EffortJointInterface</hardwareInterface>
+                <hardwareInterface>hardware_interface/VelocityJointInterface</hardwareInterface>
             </joint>
             <actuator name="wheel_5_motor">
-                <hardwareInterface>hardware_interface/EffortJointInterface</hardwareInterface>
+                <hardwareInterface>hardware_interface/VelocityJointInterface</hardwareInterface>
                 <mechanicalReduction>1</mechanicalReduction>
             </actuator>
@@ -172,5 +172,5 @@
             <parent link="drive_module_right_4_link"/>
             <child link="bogie_6_wheel"/>
-            <axis xyz="1.0 0.0 0.0"/>
+            <axis xyz="-1.0 0.0 0.0"/>
             <dynamics  damping="0.0" friction="0.5"/>
             <limit effort="30" velocity="100" />
@@ -180,8 +180,8 @@
             <type>transmission_interface/SimpleTransmission</type>
             <joint name="wheel_6_joint">
-                <hardwareInterface>hardware_interface/EffortJointInterface</hardwareInterface>
+                <hardwareInterface>hardware_interface/VelocityJointInterface</hardwareInterface>
             </joint>
             <actuator name="wheel_6_motor">
-                <hardwareInterface>hardware_interface/EffortJointInterface</hardwareInterface>
+                <hardwareInterface>hardware_interface/VelocityJointInterface</hardwareInterface>
                 <mechanicalReduction>1</mechanicalReduction>
             </actuator>
